Commit message: can make circuit demos

File: predicators/envs/assets/urdf/bulb_box_snap.urdf (robot description, URDF)
Before this commit: robot combined_bulb_box_snap_2unit, 6 links, 5 joints
Joints:
- joint end_metal_joint: origin xyz=0.07500000000000001 0 0 rpy=0 0 0 -> xyz=0.075 0 0 rpy=0 0 0
- joint line_joint: origin xyz=0 0 0.025050000000000003 rpy=0 0 0 -> xyz=0 0 0.025 rpy=0 0 0
- joint start_metal_joint: origin xyz=-0.07500000000000001 0 0 rpy=0 0 0 -> xyz=-0.075 0 0 rpy=0 0 0

File: predicators/envs/assets/urdf/snap_connector4.urdf (robot description, URDF)
Before this commit: robot snap_connector_4, 4 links, 3 joints
Links:
- link line: geometry collision box size=0.3 0.01 0.0001; visual box size=0.3 0.01 0.0001
- link middle_plastic: geometry collision box size=0.3 0.05 0.05; visual box size=0.30 0.05 0.05
Joints:
- joint end_metal_joint: origin xyz=0.17500000000000002 0 0 rpy=0 0 0 -> xyz=0.175 0 0 rpy=0 0 0
- joint line_joint: origin xyz=0 0 0.025050000000000003 rpy=0 0 0 -> xyz=0 0 0.025 rpy=0 0 0
- joint start_metal_joint: origin xyz=-0.17500000000000002 0 0 rpy=0 0 0 -> xyz=-0.1750 0 0 rpy=0 0 0
