Commit message: wip

File: predicators/envs/assets/urdf/domino_target.urdf (robot description, URDF)
Before this commit: robot simple_flap, 6 links, 5 joints
Links:
- link flap_panel: geometry collision box size=0.06 0.003 0.14; visual box size=0.06 0.003 0.14
- link left_bar: geometry collision cylinder length=0.15 radius=0.005; visual cylinder length=0.15 radius=0.005
- link middle_bar: geometry collision cylinder length=0.07 radius=0.005; visual cylinder length=0.07 radius=0.005
- link right_bar: geometry collision cylinder length=0.15 radius=0.005; visual cylinder length=0.15 radius=0.005
- link short_flap1: geometry collision box size=0.06 0.003 0.13; visual box size=0.06 0.003 0.13
- link short_flap2: geometry collision box size=0.06 0.003 0.13; visual box size=0.06 0.003 0.13
Joints:
- joint flap_hinge_joint: origin xyz=0 0 0.25 rpy=0 0 0 -> xyz=0 0 0.15 rpy=0 0 0

Commit message: update domino_target.urdf dimensions and colors for visual consistency

File: predicators/envs/assets/urdf/domino_target.urdf (robot description, URDF)
Before this commit: robot simple_flap, 6 links, 5 joints
Links:
- link flap_panel: mass 10.0 -> 0.001; geometry collision box size=0.06 0.003 0.0; visual box size=0.06 0.003 0.0
- link left_bar: geometry collision cylinder length=0.25 radius=0.005; visual cylinder length=0.25 radius=0.005
- link middle_bar: geometry collision cylinder length=0.09 radius=0.005; visual cylinder length=0.09 radius=0.005
- link right_bar: geometry collision cylinder length=0.25 radius=0.005; visual cylinder length=0.25 radius=0.005
- link short_flap1: mass 5.0 -> 0.001; geometry collision box size=0.06 0.003 0.18; visual box size=0.06 0.003 0.18
- link short_flap2: mass 5.0 -> 0.001; geometry collision box size=0.06 0.003 0.18; visual box size=0.06 0.003 0.18
Joints:
- joint flap_hinge_joint: origin xyz=0 0 0.15 rpy=0 0 0 -> xyz=0 0 0.25 rpy=0 0 0

Commit message: add pivot to domino

File: predicators/envs/assets/urdf/domino_target.urdf (robot description, URDF)
Before this commit: robot simple_flap, 6 links, 5 joints
Links:
- link flap_panel: mass 0.005 -> 0.001
- link short_flap1: mass 0.005 -> 0.001; geometry collision box size=0.06 0.003 0.15; visual box size=0.06 0.003 0.15
- link short_flap2: mass 0.005 -> 0.001; geometry collision box size=0.06 0.003 0.15; visual box size=0.06 0.003 0.15
