Commit message: make mirror narrower

File: predicators/envs/assets/urdf/laser_mirror1.urdf (robot description, URDF)
Before this commit: robot mirror_piece, 2 links, 1 joints
Links:
- link mirror_piece_body: geometry collision box size=0.07 0.01 0.1; visual box size=0.07 0.01 0.1

File: predicators/envs/assets/urdf/laser_mirror2.urdf (robot description, URDF)
Before this commit: robot mirror_piece, 2 links, 1 joints
Links:
- link mirror_piece_body: geometry collision box size=0.07 0.01 0.1; visual box size=0.07 0.01 0.1

Commit message: drop weight, add friction

File: predicators/envs/assets/urdf/laser_mirror1.urdf (robot description, URDF)
Before this commit: robot mirror_piece, 2 links, 1 joints
Links:
- link base_link: mass None -> 0.1
- link mirror_piece_body: mass None -> 0.1

File: predicators/envs/assets/urdf/laser_mirror2.urdf (robot description, URDF)
Before this commit: robot mirror_piece, 2 links, 1 joints
Links:
- link base_link: mass None -> 0.1
- link mirror_piece_body: mass None -> 0.1

Commit message: can make pick/place laser demo

File: predicators/envs/assets/urdf/laser_mirror1.urdf (robot description, URDF)
Before this commit: robot mirror_piece, 2 links, 1 joints
Links:
- link base_link: mass 0.1 -> 1
- link mirror_piece_body: mass 0.1 -> 1

File: predicators/envs/assets/urdf/laser_mirror2.urdf (robot description, URDF)
Before this commit: robot mirror_piece, 2 links, 1 joints
Links:
- link base_link: mass 0.1 -> 1
- link mirror_piece_body: mass 0.1 -> 1
