Commit message: domino video can work

File: predicators/envs/assets/urdf/domino_pivot.urdf (robot description, URDF)
Before this commit: robot horizontal_flap, 2 links, 1 joints
Links:
- link horizontal_flap: mass 0.0005 -> 0.001; geometry collision box size=0.2 0.1 0.016; visual box size=0.2 0.1 0.016
- link vertical_bar: mass 0.0005 -> 0.001
Joints:
- joint flap_hinge_joint: origin xyz=0 0 0.16 rpy=1.5707963267948966 0 0 -> xyz=0 0 0.15000000000000002 rpy=1.5707963267948966 0 0

File: predicators/envs/assets/urdf/domino_target.urdf (robot description, URDF)
Before this commit: robot simple_flap, 6 links, 5 joints
Links:
- link flap_panel: geometry collision box size=0.06 0.016 0.0; visual box size=0.06 0.016 0.0
- link short_flap1: geometry collision box size=0.06 0.016 0.15; visual box size=0.06 0.016 0.15
- link short_flap2: geometry collision box size=0.06 0.016 0.15; visual box size=0.06 0.016 0.15
Joints:
- joint short_flap1_joint: origin xyz=0 0.01 0 rpy=0.3490658503988659 0 0 -> xyz=0 0.02 0 rpy=0.2617993877991494 0 0
- joint short_flap2_joint: origin xyz=0 -0.01 0 rpy=-0.3490658503988659 0 0 -> xyz=0 -0.02 0 rpy=-0.2617993877991494 0 0
