Commit message: Basic ring env working

File: predicators/envs/assets/urdf/pole.urdf (robot description, URDF)
Before this commit: robot pole_with_base, 2 links, 1 joints
Links:
- link rod: geometry collision cylinder length=.1 radius=0.005; visual cylinder length=.1 radius=0.005

Commit message: Ring env finished and multimodal cover implemented

File: predicators/envs/assets/urdf/pole.urdf (robot description, URDF)
Before this commit: robot pole_with_base, 2 links, 1 joints
Links:
- link base: geometry collision cylinder length=0.02 radius=0.07; visual cylinder length=0.02 radius=0.07
- link rod: geometry collision cylinder length=.15 radius=0.004; visual cylinder length=.15 radius=0.004

File: predicators/envs/assets/urdf/ring.urdf (robot description, URDF)
Before this commit: robot ring, 1 links, 0 joints
Links:
- link baseLink: geometry collision mesh filename=ring.obj scale=1 1 1.85; visual mesh filename=ring.obj scale=1 1 1.85

Commit message: Finalize ring stack and multimodal cover environments

File: predicators/envs/assets/urdf/pole.urdf (robot description, URDF)
Before this commit: robot pole_with_base, 2 links, 1 joints
Links:
- link rod: geometry collision cylinder length=.15 radius=0.003; visual cylinder length=.15 radius=0.003
